Commit message: Add hardware interface for Real Robot and Modify URDF

File: description/camera.xacro (robot description, xacro)
@@ -5,25 +5,18 @@
         <parent link="chassis"/>
         <child link="camera_link"/>
-        <origin xyz="0.09 0 0.11"/>
+        <origin xyz="0.08 0 0.17"/>
     </joint>
     <link name="camera_link">
         <visual>
-            <origin xyz="0 0 0"/>
+            <origin xyz="0 0 -0.01" rpy = "0 0 ${-pi/2}"/>
             <geometry>
-                <box size="0.02 0.025 0.025"/>
+                <mesh filename="file:///$(find dhtbot_one)/meshes/intel_realsense_D435.stl" scale="0.001 0.001 0.001"/>
             </geometry>
-            <material name="orange"/>
-        </visual>
-        <visual>
-            <origin xyz="0.015 0 0" rpy="0 ${pi/2} 0"/>
-            <geometry>
-                <cylinder radius="0.0075" length="0.01"/>
-            </geometry>
-            <material name="orange"/>
+            <material name="gray"/>
         </visual>
         <collision>
-            <origin xyz="0.01 0 0"/>
+            <origin xyz="0 0 0" />
             <geometry>
-                <box size="0.03 0.025 0.025"/>
+                <box size="0.03 0.08 0.03"/>
             </geometry>
         </collision>

File: description/gazebo_control.xacro (robot description, xacro)
@@ -6,8 +6,8 @@
             <left_joint>left_wheel_joint</left_joint>
             <right_joint>right_wheel_joint</right_joint>
-            <wheel_separation>0.35</wheel_separation>
-            <wheel_diameter>0.1</wheel_diameter>
+            <wheel_separation>0.175</wheel_separation>
+            <wheel_diameter>0.0325</wheel_diameter>
             <!-- Limits -->
-            <max_wheel_torque>200</max_wheel_torque>
+            <max_wheel_torque>5</max_wheel_torque>
             <max_wheel_acceleration>1.5</max_wheel_acceleration>
             <!-- Output -->
@@ -17,4 +17,7 @@
             <publish_odom_tf>true</publish_odom_tf>
             <publish_wheel_tf>true</publish_wheel_tf>
+            <ros>
+                <namespace>/robot</namespace>
+            </ros>
         </plugin>
     </gazebo>

File: description/robot.urdf.xacro (robot description, xacro)
@@ -1,4 +1,5 @@
 <?xml version="1.0"?>
 <robot xmlns:xacro="http://www.ros.org/wiki/xacro"  name="robot">
+    <xacro:arg name="sim_mode" default="false"/>
     <xacro:include filename="robot_core.xacro" />
     <!-- <xacro:include filename="gazebo_control.xacro" /> -->

File: description/robot_core.xacro (robot description, xacro)
@@ -28,9 +28,7 @@
     <link name="chassis">
         <visual>
-            <origin xyz="0 0 -0.015"/>
-            <!--<origin xyz="0 0 0.045"/>-->
+            <origin xyz="0 0 -0.014" rpy="0 0 ${pi}"/>
             <geometry>
-                <mesh filename="file:///$(find dhtbot_one)/meshes/base_link.STL" scale="1 1 1"/>-->
-                <!--<cylinder radius="0.115" length="0.12"/>-->
+                <mesh filename="file:///$(find dhtbot_one)/meshes/base_link.STL" scale="1 1 1"/>
             </geometry>
             <material name="white"/>
@@ -65,10 +63,10 @@
         <collision>
             <geometry>
-                <cylinder radius="0.0325" length="0.025"/>
+                <sphere radius="0.0325"/>
             </geometry>
         </collision>
-        <xacro:inertial_cylinder mass="0.1" length="0.025" radius="0.0325">
+        <xacro:inertial_sphere mass="0.1" radius="0.0325">
             <origin xyz="0 0 0" rpy="0 0 0"/>
-        </xacro:inertial_cylinder>
+        </xacro:inertial_sphere>
     </link>
     <gazebo reference="left_wheel">
@@ -93,10 +91,10 @@
         <collision>
             <geometry>
-                <cylinder radius="0.0325" length="0.025"/>
+                <sphere radius="0.0325"/>
             </geometry>
         </collision>
-        <xacro:inertial_cylinder mass="0.1" length="0.025" radius="0.0325">
+        <xacro:inertial_sphere mass="0.1" radius="0.0325">
             <origin xyz="0 0 0" rpy="0 0 0"/>
-        </xacro:inertial_cylinder>
+        </xacro:inertial_sphere>
     </link>
     <gazebo reference="right_wheel">

File: description/ros2_control.xacro (robot description, xacro)
@@ -1,28 +1,54 @@
 <?xml version="1.0"?>
 <robot xmlns:xacro="http://www.ros.org/wiki/xacro">
-    <ros2_control name="GazeboSystem" type="system">
-        <hardware>
-            <plugin>gazebo_ros2_control/GazeboSystem</plugin>
-        </hardware>
-        <joint name="left_wheel_joint">
-            <command_interface name="velocity">
-                <param name="min">-5</param>
-                <param name="max">5</param>
-            </command_interface>
-            <state_interface name="velocity"/>
-            <state_interface name="position"/>
-        </joint>
-        <joint name="right_wheel_joint">
-            <command_interface name="velocity">
-                <param name="min">-5</param>
-                <param name="max">5</param>
-            </command_interface>
-            <state_interface name="velocity"/>
-            <state_interface name="position"/>
-        </joint>
-    </ros2_control>
+    <xacro:unless value="$(arg sim_mode)">
+        <ros2_control name="RealRobot" type="system">
+            <hardware>
+                <plugin>diffbot_system_hardware/DiffBotSystemHardware</plugin>
+                <param name="left_wheel_name">left_wheel_joint</param>
+                <param name="right_wheel_name">right_wheel_joint</param>
+                <param name="device">/dev/ttyUSB0</param>
+                <param name="baud_rate">115200</param>
+                <param name="timeout_ms">1000</param>
+                <param name="enc_counts_per_rev">7400</param>
+            </hardware>
+            <joint name="left_wheel_joint">
+                <command_interface name="velocity"/>
+                <state_interface name="position"/>
+                <state_interface name="velocity"/>
+            </joint>
+            <joint name="right_wheel_joint">
+                <command_interface name="velocity"/>
+                <state_interface name="position"/>
+                <state_interface name="velocity"/>
+            </joint>
+        </ros2_control>
+    </xacro:unless>
+    <xacro:if value="$(arg sim_mode)">
+        <ros2_control name="GazeboSystem" type="system">
+            <hardware>
+                <plugin>gazebo_ros2_control/GazeboSystem</plugin>
+            </hardware>
+            <joint name="left_wheel_joint">
+                <command_interface name="velocity">
+                    <param name="min">-10</param>
+                    <param name="max">10</param>
+                </command_interface>
+                <state_interface name="velocity"/>
+                <state_interface name="position"/>
+            </joint>
+            <joint name="right_wheel_joint">
+                <command_interface name="velocity">
+                    <param name="min">-10</param>
+                    <param name="max">10</param>
+                </command_interface>
+                <state_interface name="velocity"/>
+                <state_interface name="position"/>
+            </joint>
+        </ros2_control>
+    </xacro:if>
     <gazebo>
         <plugin name="gazebo_ros2_control" filename="libgazebo_ros2_control.so">
             <parameters>$(find dhtbot_one)/config/my_controllers.yaml</parameters>
+            <parameters>$(find dhtbot_one)/config/gazebo_use_sim_time.yaml</parameters>
         </plugin>
     </gazebo>
